Commit message: changes

File: my_sdfs/panda_hand.urdf (robot description, URDF)
Before this commit: robot panda_hand, 4 links, 3 joints
Joints:
- joint panda_finger_joint2: axis 0 1 0 -> (none); limit lower=0.0 upper=0.045 effort=20 velocity=0.2 -> (none); type prismatic -> fixed

Commit message: Lock Panda grasp joints for reduced C-space

File: my_sdfs/panda_hand.urdf (robot description, URDF)
Before this commit: robot panda_hand, 4 links, 3 joints
Joints:
- joint panda_finger_joint2: origin xyz=0 0 0.0584 rpy=0 0 0 -> xyz=0 0.024 0.0584 rpy=0 0 0
