Commit message: updates in debugging version error of GCS

File: my_sdfs/panda_hand_locked.urdf (robot description, URDF)
Before this commit: robot panda_hand, 4 links, 3 joints
Joints:
- joint panda_finger_joint2: axis 0 1 0 -> (none); limit lower=0.0 upper=0.045 effort=20 velocity=0.2 -> (none); origin xyz=0 0 0.0584 rpy=0 0 0 -> xyz=0 0.026 0.0584 rpy=0 0 0; type prismatic -> fixed
